Commit message: fixed urdf and lauch file for rviz and gazebo

File: autonav_description/urdf/autonav.xacro (robot description, xacro)
@@ -30,5 +30,5 @@
   </inertial>
   <visual>
-    <origin xyz="-0.15 0.0 -0.082" rpy="0 0 0"/>
+    <origin xyz="-0.175 0.0 -0.082" rpy="0 0 0"/>
     <geometry>
       <mesh filename="package://autonav_description/meshes/depth_camera_1.stl" scale="0.001 0.001 0.001"/>
@@ -37,5 +37,5 @@
   </visual>
   <collision>
-    <origin xyz="-0.15 0.0 -0.082" rpy="0 0 0"/>
+    <origin xyz="-0.175 0.0 -0.082" rpy="0 0 0"/>
     <geometry>
       <mesh filename="package://autonav_description/meshes/depth_camera_1.stl" scale="0.001 0.001 0.001"/>
@@ -90,5 +90,5 @@
   </inertial>
   <visual>
-    <origin xyz="-0.063 -0.025 -0.1515" rpy="0 0 0"/>
+    <origin xyz="-0.0955 -0.0 -0.196" rpy="0 0 0"/>
     <geometry>
       <mesh filename="package://autonav_description/meshes/lidar_1.stl" scale="0.001 0.001 0.001"/>
@@ -97,5 +97,5 @@
   </visual>
   <collision>
-    <origin xyz="-0.063 -0.025 -0.1515" rpy="0 0 0"/>
+    <origin xyz="-0.0955 -0.0 -0.196" rpy="0 0 0"/>
     <geometry>
       <mesh filename="package://autonav_description/meshes/lidar_1.stl" scale="0.001 0.001 0.001"/>
@@ -123,10 +123,10 @@
   </collision>
 </link>
-<joint name="Rigid 16" type="fixed">
-  <origin xyz="0.15 0.0 0.082" rpy="0 0 0"/>
+<joint name="base2depth" type="fixed">
+  <origin xyz="0.175 0.0 0.082" rpy="0 0 0"/>
   <parent link="base_link"/>
   <child link="depth_camera_1"/>
 </joint>
-<joint name="Revolute 17" type="continuous">
+<joint name="base2right" type="continuous">
   <origin xyz="-0.00075 -0.105044 0.04" rpy="0 0 0"/>
   <parent link="base_link"/>
@@ -134,5 +134,5 @@
   <axis xyz="-0.0 -1.0 0.0"/>
 </joint>
-<joint name="Revolute 18" type="continuous">
+<joint name="base2left" type="continuous">
   <origin xyz="-0.00075 0.105 0.04" rpy="0 0 0"/>
   <parent link="base_link"/>
@@ -140,10 +140,10 @@
   <axis xyz="0.0 1.0 -0.0"/>
 </joint>
-<joint name="Rigid 19" type="fixed">
-  <origin xyz="0.063 0.025 0.1515" rpy="0 0 0"/>
+<joint name="base2lidar" type="fixed">
+  <origin xyz="0.0955 0.0 0.196" rpy="0 0 0"/>
   <parent link="base_link"/>
   <child link="lidar_1"/>
 </joint>
-<joint name="Rigid 20" type="fixed">
+<joint name="base2imu" type="fixed">
   <origin xyz="0.0675 0.05 0.0835" rpy="0 0 0"/>
   <parent link="base_link"/>

File: autonav_description/urdf/materials.xacro (robot description, xacro)
@@ -14,8 +14,8 @@
 </material>
 <material name="paint_enamel_glossy_grey">
-  <color rgba="0.7019607843137254 0.7019607843137254 0.7019607843137254 0.0"/>
+  <color rgba="0.7019607843137254 0.7019607843137254 0.7019607843137254 1.0"/>
 </material>
 <material name="powder_coat_grey">
-  <color rgba="0.7019607843137254 0.7019607843137254 0.7019607843137254 0.0"/>
+  <color rgba="0.7019607843137254 0.7019607843137254 0.7019607843137254 1.0"/>
 </material>
 </robot>

Commit message: Updated controllers

File: autonav_description/urdf/autonav.xacro (robot description, xacro)
@@ -4,4 +4,5 @@
 <xacro:include filename="$(find autonav_description)/urdf/autonav_gazebo.xacro" />
 <xacro:include filename="$(find autonav_description)/urdf/autonav_ros2_control.xacro" />
+<link name="base_footprint"/>
 <link name="base_link">
   <inertial>
@@ -18,10 +19,21 @@
   </visual>
   <collision>
-    <origin xyz="0 0 0" rpy="0 0 0"/>
+    <!-- <origin xyz="0 0 0" rpy="0 0 0"/>
     <geometry>
       <mesh filename="package://autonav_description/meshes/base_link.stl" scale="0.001 0.001 0.001"/>
+    </geometry> -->
+    <origin xyz="0.04 0 0.005" rpy="0 0 0"/>
+    <geometry>
+      <!-- <mesh filename="package://cube_description/meshes/base_link.stl" scale="0.001 0.001 0.001"/> -->
+      <box size="0.20 0.18 0.01" />
     </geometry>
   </collision>
 </link>
+<joint name="footprint2baselink" type="fixed">
+  <parent link="base_footprint"/>
+  <child link="base_link"/>
+  <origin xyz="0 0 0" rpy="0 0 0"/>
+  <axis xyz="0 0 0"/>
+</joint>
 <link name="depth_camera_1">
   <inertial>
@@ -130,8 +142,8 @@
 </joint>
 <joint name="base2right" type="continuous">
-  <origin xyz="-0.00075 -0.105044 0.04" rpy="0 0 0"/>
+  <origin xyz="-0.00075 -0.105 0.04" rpy="0 0 0"/>
   <parent link="base_link"/>
   <child link="right_wheel_1"/>
-  <axis xyz="-0.0 -1.0 0.0"/>
+  <axis xyz="-0.0 1.0 0.0"/>
 </joint>
 <joint name="base2left" type="continuous">

File: autonav_description/urdf/autonav_gazebo.xacro (robot description, xacro)
@@ -43,4 +43,28 @@
     <maxVel>1.0</maxVel>
   </gazebo>
+  <gazebo reference="depth_camera_1">
+    <mu1>0.1</mu1>
+    <mu2>0.1</mu2>
+    <kp>1000000.0</kp>
+    <kd>100.0</kd>
+    <minDepth>0.001</minDepth>
+    <maxVel>1.0</maxVel>
+  </gazebo>
+  <gazebo reference="lidar_1">
+    <mu1>0.1</mu1>
+    <mu2>0.1</mu2>
+    <kp>1000000.0</kp>
+    <kd>100.0</kd>
+    <minDepth>0.001</minDepth>
+    <maxVel>1.0</maxVel>
+  </gazebo>
+  <gazebo reference="imu_1">
+    <mu1>0.1</mu1>
+    <mu2>0.1</mu2>
+    <kp>1000000.0</kp>
+    <kd>100.0</kd>
+    <minDepth>0.001</minDepth>
+    <maxVel>1.0</maxVel>
+  </gazebo>
   <!-- ROS 2 Control -->
   <gazebo>

Commit message: Changed Camera link in urdf

File: autonav_description/urdf/autonav.xacro (robot description, xacro)
@@ -36,5 +36,5 @@
   <axis xyz="0 0 0"/>
 </joint>
-<link name="depth_camera_1">
+<link name="camera_link">
   <inertial>
     <origin xyz="0.013571033223507722 -1.5421816108169115e-15 -1.8457457784393227e-15" rpy="0 0 0"/>
@@ -139,5 +139,5 @@
   <origin xyz="0.175 0.0 0.082" rpy="0 0 0"/>
   <parent link="base_link"/>
-  <child link="depth_camera_1"/>
+  <child link="camera_link"/>
 </joint>
 <joint name="base2right" type="continuous">

Commit message: Added gazebo pkg and launch file

File: autonav_description/urdf/autonav.xacro (robot description, xacro)
@@ -3,5 +3,4 @@
 <xacro:include filename="$(find autonav_description)/urdf/materials.xacro" />
 <xacro:include filename="$(find autonav_description)/urdf/autonav_gazebo.xacro" />
-<xacro:include filename="$(find autonav_description)/urdf/autonav_ros2_control.xacro" />
 <link name="base_footprint"/>
 <link name="base_link">
@@ -16,5 +15,5 @@
       <mesh filename="package://autonav_description/meshes/base_link.stl" scale="0.001 0.001 0.001"/>
     </geometry>
-    <material name="powder_coat_grey"/>
+    <material name="black"/>
   </visual>
   <collision>
@@ -56,4 +55,11 @@
   </collision>
 </link>
+<link name="camera_link_1"/>
+<joint name="camera2camera_1" type="fixed">
+  <parent link="camera_link"/>
+  <child link="camera_link_1"/>
+  <origin xyz="0 0 0" rpy="-1.5708 0 -1.5708"/>
+  <axis xyz="0 0 0"/>
+</joint>
 <link name="right_wheel_1">
   <inertial>
@@ -107,5 +113,5 @@
       <mesh filename="package://autonav_description/meshes/lidar_1.stl" scale="0.001 0.001 0.001"/>
     </geometry>
-    <material name="steel_satin"/>
+    <material name="blue"/>
   </visual>
   <collision>

File: autonav_description/urdf/autonav_gazebo.xacro (robot description, xacro)
@@ -1,4 +1,9 @@
 <?xml version="1.0"?>
 <robot name="autonav" xmlns:xacro="http://ros.org/wiki/xacro">
+<xacro:property name="base_link" value="Gazebo/FlatBlack" />
+<xacro:property name="wheels" value="Gazebo/Black" />
+<xacro:property name="imu" value="Gazebo/PurpleGlow" />
+<xacro:property name="lidar" value="Gazebo/BlueGlow" />
+<xacro:property name="depth_cam" value="Gazebo/TurquoiseGlow" />
   <transmission name="wheel_right_transmission">
     <plugin>transmission_interface/SimpleTransmission</plugin>
@@ -17,4 +22,5 @@
   <!-- Wheels -->
   <gazebo reference="left_wheel_1">
+    <material>${wheels}</material>
     <mu1>1000000000000000.0</mu1>
     <mu2>1000000000000000.0</mu2>
@@ -26,4 +32,5 @@
   </gazebo>
   <gazebo reference="right_wheel_1">
+    <material>${wheels}</material>
     <mu1>1000000000000000.0</mu1>
     <mu2>1000000000000000.0</mu2>
@@ -36,12 +43,14 @@
   <!-- Caster Wheels -->
   <gazebo reference="base_link">
-    <mu1>0.1</mu1>
-    <mu2>0.1</mu2>
-    <kp>1000000.0</kp>
-    <kd>100.0</kd>
-    <minDepth>0.001</minDepth>
-    <maxVel>1.0</maxVel>
-  </gazebo>
-  <gazebo reference="depth_camera_1">
+    <material>${base_link}</material>
+    <mu1>0.1</mu1>
+    <mu2>0.1</mu2>
+    <kp>1000000.0</kp>
+    <kd>100.0</kd>
+    <minDepth>0.001</minDepth>
+    <maxVel>1.0</maxVel>
+  </gazebo>
+  <gazebo reference="camera_link">
+    <material>${depth_cam}</material>
     <mu1>0.1</mu1>
     <mu2>0.1</mu2>
@@ -52,4 +61,5 @@
   </gazebo>
   <gazebo reference="lidar_1">
+    <material>${lidar}</material>
     <mu1>0.1</mu1>
     <mu2>0.1</mu2>
@@ -60,18 +70,155 @@
   </gazebo>
   <gazebo reference="imu_1">
-    <mu1>0.1</mu1>
-    <mu2>0.1</mu2>
-    <kp>1000000.0</kp>
-    <kd>100.0</kd>
-    <minDepth>0.001</minDepth>
-    <maxVel>1.0</maxVel>
-  </gazebo>
-  <!-- ROS 2 Control -->
+    <material>${imu}</material>
+    <mu1>0.1</mu1>
+    <mu2>0.1</mu2>
+    <kp>1000000.0</kp>
+    <kd>100.0</kd>
+    <minDepth>0.001</minDepth>
+    <maxVel>1.0</maxVel>
+  </gazebo>
   <gazebo>
-    <plugin filename="libgazebo_ros2_control.so" name="gazebo_ros2_control">
-      <robot_param>robot_description</robot_param>
-      <robot_param_node>robot_state_publisher</robot_param_node>
-      <parameters>$(find autonav_controller)/config/autonav_controllers.yaml</parameters>
+    <plugin name="diff_drive_control" filename="libgazebo_ros_diff_drive.so">
+      <!-- Update rate in Hz -->
+      <update_rate>50</update_rate>
+      <!-- wheels -->
+      <left_joint>base2left</left_joint>
+      <right_joint>base2right</right_joint>
+      <!-- kinematics -->
+      <wheel_separation>0.21</wheel_separation>
+      <wheel_diameter>0.08</wheel_diameter>
+      <!-- input -->
+      <command_topic>cmd_vel</command_topic>
+      <!-- output -->
+      <publish_odom>true</publish_odom>
+      <publish_odom_tf>true</publish_odom_tf>
+      <publish_wheel_tf>true</publish_wheel_tf>
+      <odometry_topic>odom</odometry_topic>
+      <odometry_frame>odom</odometry_frame>
+      <robot_base_frame>base_footprint</robot_base_frame>
     </plugin>
   </gazebo>
+  <gazebo reference="imu_1">
+    <gravity>true</gravity>
+    <sensor name="imu_1" type="imu">
+      <always_on>true</always_on>
+      <update_rate>30</update_rate>
+      <visualize>true</visualize>
+      <plugin name="my_imu_plugin" filename="libgazebo_ros_imu_sensor.so">
+        <ros>
+          <remapping>~/out:=imu</remapping>
+        </ros>
+        <frame_name>imu_1</frame_name>
+      </plugin>
+    </sensor>
+  </gazebo>
+  <gazebo reference="lidar_1">
+    <sensor type="ray" name="head_hokuyo_sensor">
+      <pose>0 0 0 0 0 0</pose>
+      <visualize>false</visualize>
+      <update_rate>30</update_rate>
+      <ray>
+        <scan>
+          <horizontal>
+            <samples>300</samples>
+            <resolution>1</resolution>
+            <min_angle>-3.14</min_angle>
+            <max_angle>3.14</max_angle>
+          </horizontal>
+        </scan>
+        <range>
+          <min>0.10</min>
+          <max>30.0</max>
+          <resolution>0.01</resolution>
+        </range>
+        <noise>
+          <type>gaussian</type>
+          <!-- Noise parameters based on published spec for Hokuyo laser
+               achieving "+-30mm" accuracy at range < 10m.  A mean of 0.0m and
+               stddev of 0.01m will put 99.7% of samples within 0.03m of the true
+               reading. -->
+          <mean>0.0</mean>
+          <stddev>0.01</stddev>
+        </noise>
+      </ray>
+      <plugin name="my_ray_sensor_plugin" filename="libgazebo_ros_ray_sensor.so">
+        <ros>
+          <!-- Configure namespace and remap to publish to /ray/pointcloud2 -->
+          <remapping>~/out:=scan</remapping>
+        </ros>
+        <!-- Output as a PointCloud2, see above for other types -->
+        <output_type>sensor_msgs/LaserScan</output_type>
+        <!-- Clip intensity values so all are above 100, optional -->
+        <min_intensity>100.0</min_intensity>
+        <!-- Frame id for header of output, defaults to sensor's parent link name -->
+        <frame_name>lidar_1</frame_name>
+      </plugin>
+    </sensor>
+  </gazebo>
+  <gazebo reference="camera_link">
+    <sensor name="camera" type="depth">
+      <pose> 0 0 0 0 0 0</pose>
+      <visualize>true</visualize>
+      <update_rate>60.0</update_rate>
+      <camera name="camera_link">
+        <horizontal_fov>1.047198</horizontal_fov>
+        <image>
+          <width>640</width>
+          <height>480</height>
+          <format>R8G8B8</format>
+        </image>
+        <clip>
+          <near>0.05</near>
+          <far>10</far>
+        </clip>
+      </camera>
+      <plugin name="depth_camera_controller" filename="libgazebo_ros_camera.so">
+        <!-- <ros>
+          <remapping>/camera/camera_info:=/camera/rgb/camera_info</remapping>
+          <remapping>/camera/image_raw:=/camera/rgb/image_rect_color</remapping>
+          <remapping>/camera/depth/image_raw:=/camera/depth_registered/image_raw</remapping>
+        </ros> -->
+        <baseline>0.2</baseline>
+        <alwaysOn>true</alwaysOn>
+        <updateRate>0.0</updateRate>
+        <frame_name>camera_link_1</frame_name>
+        <pointCloudCutoff>0.1</pointCloudCutoff>
+        <pointCloudCutoffMax>10.0</pointCloudCutoffMax>
+        <distortionK1>0</distortionK1>
+        <distortionK2>0</distortionK2>
+        <distortionK3>0</distortionK3>
+        <distortionT1>0</distortionT1>
+        <distortionT2>0</distortionT2>
+        <CxPrime>0</CxPrime>
+        <Cx>0</Cx>
+        <Cy>0</Cy>
+        <focalLength>0</focalLength>
+        <hackBaseline>0</hackBaseline>
+      </plugin>
+      <!-- <plugin name="camera_plugin" filename="libgazebo_ros_camera.so">
+        <baseline>0.2</baseline>
+        <alwaysOn>true</alwaysOn>
+        <updateRate>0.0</updateRate>
+        <cameraName>camera_ir</cameraName>
+        <imageTopicName>/camera/color/image_raw</imageTopicName>
+        <cameraInfoTopicName>/camera/color/camera_info</cameraInfoTopicName>
+        <depthImageTopicName>/camera/depth/image_raw</depthImageTopicName>
+        <depthImageCameraInfoTopicName>/camera/depth/camera_info</depthImageCameraInfoTopicName>
+        <pointCloudTopicName>/camera/depth/points</pointCloudTopicName>
+        <frameName>camera_link</frameName>
+        <pointCloudCutoff>0.5</pointCloudCutoff>
+        <pointCloudCutoffMax>3.0</pointCloudCutoffMax>
+        <distortionK1>0</distortionK1>
+        <distortionK2>0</distortionK2>
+        <distortionK3>0</distortionK3>
+        <distortionT1>0</distortionT1>
+        <distortionT2>0</distortionT2>
+        <CxPrime>0</CxPrime>
+        <Cx>0</Cx>
+        <Cy>0</Cy>
+        <focalLength>0</focalLength>
+        <hackBaseline>0</hackBaseline>
+      </plugin> -->
+    </sensor>
+  </gazebo>
 </robot>

File: autonav_description/urdf/materials.xacro (robot description, xacro)
@@ -19,3 +19,9 @@
   <color rgba="0.7019607843137254 0.7019607843137254 0.7019607843137254 1.0"/>
 </material>
+<material name="blue">
+  <color rgba="0.1 0.1 0.7 1.0"/>
+</material>
+<material name="black">
+  <color rgba="0.4 0.35 0.38 1.0"/>
+</material>
 </robot>

Commit message: Refactor navigation parameters and improve performance
- Updated AMCL parameters for better localization accuracy, including adjustments to alpha values, laser range, and particle counts.
- Enhanced BT navigator settings for improved behavior tree execution time.
- Modified controller server parameters to refine movement tolerances and goal checking.
- Switched from DWB to Regulated Pure Pursuit controller for path following, optimizing velocity and lookahead settings.
- Increased local and global costmap dimensions and adjusted footprint for better obstacle avoidance.
- Removed deprecated perception package, consolidating camera publishing and subscribing functionalities.
- Updated BNO055 parameters for improved sensor calibration and data query frequency.
- Adjusted Docker Compose configurations for streamlined service launches and device mappings.
- Changed YDLIDAR parameters to enable single channel and increased frequency for better data acquisition.

File: autonav_description/urdf/autonav.xacro (robot description, xacro)
@@ -159,5 +159,5 @@
 </joint>
 <joint name="base2imu" type="fixed">
-  <origin xyz="0.0675 0.05 0.0835" rpy="0 0 0"/>
+  <origin xyz="0.0675 -0.08 0.0835" rpy="0 0 0"/>
   <parent link="base_link"/>
   <child link="imu_1"/>
